Commit message: ros2 humble description

File: src/limo_description/urdf/limo_steering_hinge.xacro (robot description, xacro)
@@ -38,5 +38,5 @@
               <origin xyz="0 0 0" rpy="0 0 0" />
               <geometry>
-                  <mesh filename="package://limo_description/meshes/limo_wheel.dae" />
+                  <mesh filename="file://$(find limo_description)/meshes/limo_wheel.dae" />
               </geometry>
           </visual>
@@ -92,5 +92,5 @@
               <origin xyz="0 0 0" rpy="0 0 0" />
               <geometry>
-                  <mesh filename="package://limo_description/meshes/limo_wheel.dae" />
+                  <mesh filename="file://$(find limo_description)/meshes/limo_wheel.dae" />
               </geometry>
           </visual>

File: src/limo_description/urdf/limo_xacro.xacro (robot description, xacro)
@@ -11,5 +11,5 @@
                 <origin xyz="0 0 0" rpy="0 0 0" />
                 <geometry>
-                    <mesh filename="package://limo_description/meshes/limo_wheel.dae" />
+                    <mesh filename="file://$(find limo_description)/meshes/limo_wheel.dae" />
                 </geometry>
             </visual>
