Commit message: fixed rviz and cleaned limo_description

File: src/limo_pkgs/limo_description/urdf/limo_four_diff.xacro (robot description, xacro)
@@ -54,5 +54,5 @@
     </xacro:limo_laser>
     <xacro:limo_depth_camera parent_prefix="base_link" frame_prefix="depth_camera">
-        <origin xyz="0.084 0 0.3" rpy="0 0 0"/>
+        <origin xyz="0.084 0 0.03" rpy="0 0 0"/>
     </xacro:limo_depth_camera>
     <xacro:limo_imu parent_prefix="base_link" frame_prefix="imu">
