Commit message: fixed xacro creation for multiple robot, now senors works

File: src/limo_pkgs/limo_description/urdf/limo.xacro (robot description, xacro)
@@ -1,4 +1,4 @@
 <?xml version="1.0"?>
-<robot name="limo_xacro" xmlns:xacro="http://ros.org/wiki/xacro">
+<robot name="limo" xmlns:xacro="http://ros.org/wiki/xacro">
     <xacro:macro name="limo_wheel" params="parent_prefix wheel_prefix reflect *joint_pose">
         <link name="${wheel_prefix}_wheel_link">
@@ -92,10 +92,4 @@
             <parent link="${parent_prefix}"/>
         </joint>
-        <link name="depth_link"></link>
-        <joint name="${frame_prefix}_to_camera_joint" type="fixed">
-            <origin xyz="0 0 0" rpy="${-M_PI/2} 0 ${-M_PI/2} "/>
-            <parent link="${frame_prefix}_link"/>
-            <child link="depth_link"/>
-          </joint>
         <gazebo reference="${frame_prefix}_link">
             <material>Gazebo/Yellow</material>

File: src/limo_pkgs/limo_description/urdf/limo_four_diff.xacro (robot description, xacro)
@@ -1,5 +1,7 @@
 <?xml version="1.0"?>
-<robot name="limo_four_diff" xmlns:xacro="http://ros.org/wiki/xacro">
-    <xacro:include filename="$(find limo_description)/urdf/limo_xacro.xacro" />
+<robot name="limo" xmlns:xacro="http://ros.org/wiki/xacro">
+    <xacro:arg name="robot_id" default="" />
+    <xacro:macro name="limo" params='robot_id'>
+    <xacro:include filename="$(find limo_description)/urdf/limo.xacro" />
     <!-- Variables -->
     <xacro:property name="M_PI" value="3.14159"/>
@@ -14,12 +16,12 @@
     <xacro:property name="wheel_length" value="0.045" />
     <xacro:property name="wheel_radius" value="0.045" />
-  <link name="base_footprint"/>
-  <joint name="base_joint" type="fixed">
-    <parent link="base_footprint"/>
-    <child link="base_link"/>
+  <link name="limo${robot_id}/base_footprint"/>
+  <joint name="limo${robot_id}/base_joint" type="fixed">
+    <parent link="limo${robot_id}/base_footprint"/>
+    <child link="limo${robot_id}/base_link"/>
     <origin xyz="0.0 0.0 0.15" rpy="0 0 0"/>
   </joint>
     <!-- Base link -->
-    <link name="base_link">
+    <link name="limo${robot_id}/base_link">
         <visual>
             <origin xyz="0 0 -0.15" rpy="0 0 1.57" />
@@ -36,5 +38,5 @@
         </collision>
     </link>
-    <link name="inertial_link">
+    <link name="limo${robot_id}/inertial_link">
         <inertial>
             <origin xyz="0.0 0.0 0.0" />
@@ -45,31 +47,31 @@
         </inertial>
     </link>
-    <joint name="inertial_joint" type="fixed">
+    <joint name="limo${robot_id}/inertial_joint" type="fixed">
         <origin xyz="0 0 0" rpy="0 0 0" />
-        <parent link="base_link" />
-        <child link="inertial_link" />
+        <parent link="limo${robot_id}/base_link" />
+        <child link="limo${robot_id}/inertial_link" />
     </joint>
-    <xacro:limo_laser parent_prefix="base_link" frame_prefix="laser">
+    <xacro:limo_laser parent_prefix="limo${robot_id}/base_link" frame_prefix="limo${robot_id}/laser">
         <origin xyz="0.103 0 -0.034" rpy="0 0 0"/>
     </xacro:limo_laser>
-    <xacro:limo_depth_camera parent_prefix="base_link" frame_prefix="depth_camera">
+    <xacro:limo_depth_camera parent_prefix="limo${robot_id}/base_link" frame_prefix="limo${robot_id}/depth_camera">
         <origin xyz="0.084 0 0.03" rpy="0 0 0"/>
     </xacro:limo_depth_camera>
-    <xacro:limo_imu parent_prefix="base_link" frame_prefix="imu">
+    <xacro:limo_imu parent_prefix="limo${robot_id}/base_link" frame_prefix="limo${robot_id}/imu">
         <origin xyz="0.0 0 -0.1" rpy="0 0 0"/>
     </xacro:limo_imu>
-    <xacro:limo_wheel parent_prefix="base_link" wheel_prefix="front_left" reflect="1">
+    <xacro:limo_wheel parent_prefix="limo${robot_id}/base_link" wheel_prefix="limo${robot_id}/front_left" reflect="1">
         <origin xyz="${wheelbase/2} ${track/2} ${wheel_vertical_offset}" rpy="0 0  0" />
     </xacro:limo_wheel>
-    <xacro:limo_wheel parent_prefix="base_link" wheel_prefix="front_right" reflect="-1">
+    <xacro:limo_wheel parent_prefix="limo${robot_id}/base_link" wheel_prefix="limo${robot_id}/front_right" reflect="-1">
         <origin xyz="${wheelbase/2} ${-track/2} ${wheel_vertical_offset}" rpy="${M_PI} 0 0" />
     </xacro:limo_wheel>
-    <xacro:limo_wheel parent_prefix="base_link" wheel_prefix="rear_left" reflect="1">
+    <xacro:limo_wheel parent_prefix="limo${robot_id}/base_link" wheel_prefix="limo${robot_id}/rear_left" reflect="1">
         <origin xyz="${-wheelbase/2} ${track/2} ${wheel_vertical_offset}" rpy="0 0 0" />
     </xacro:limo_wheel>
-    <xacro:limo_wheel parent_prefix="base_link" wheel_prefix="rear_right" reflect="-1">
+    <xacro:limo_wheel parent_prefix="limo${robot_id}/base_link" wheel_prefix="limo${robot_id}/rear_right" reflect="-1">
         <origin xyz="${-wheelbase/2} ${-track/2} ${wheel_vertical_offset}" rpy="${M_PI} 0 0" />
     </xacro:limo_wheel>
-    <gazebo reference="imu_link">
+    <gazebo reference="limo${robot_id}/imu_link">
     <gravity>true</gravity>
     <sensor name="twr_imu" type="imu">
@@ -141,5 +143,5 @@
       <plugin name="two_wheeled_robot_imu" filename="libgazebo_ros_imu_sensor.so">
         <initial_orientation_as_reference>false</initial_orientation_as_reference>
-        <frame_name>imu_link</frame_name>
+        <frame_name>limo${robot_id}/imu_link</frame_name>
         <ros>
           <remapping>~/out:=data</remapping>
@@ -148,5 +150,5 @@
     </sensor>
 </gazebo>
-<gazebo reference="laser_link">
+<gazebo reference="limo${robot_id}/laser_link">
     <sensor name="laser" type="ray">
       <always_on>true</always_on>
@@ -178,36 +180,36 @@
         </ros>
         <output_type>sensor_msgs/LaserScan</output_type>
-        <frame_name>laser_link</frame_name>
+        <frame_name>limo${robot_id}/laser_link</frame_name>
       </plugin>
     </sensor>
   </gazebo>
-    <gazebo reference="front_left_wheel">
-        <mu1>100</mu1>
-        <mu2>100</mu2>
-        <kp>10000000.0</kp>
-        <kd>1.0</kd>
-        <minDepth>0.01</minDepth>
-        <fdir1>1 0 0</fdir1>
-        <maxContacts value="64"/>
-    </gazebo>
-    <gazebo reference="front_right_wheel">
-        <mu1>100</mu1>
-        <mu2>100</mu2>
-        <kp>10000000.0</kp>
-        <kd>1.0</kd>
-        <minDepth>0.01</minDepth>
-        <fdir1>1 0 0</fdir1>
-        <maxContacts value="64"/>
-    </gazebo>
-    <gazebo reference="rear_left_wheel">
-        <mu1>100</mu1>
-        <mu2>100</mu2>
-        <kp>10000000.0</kp>
-        <kd>1.0</kd>
-        <minDepth>0.01</minDepth>
-        <fdir1>1 0 0</fdir1>
-        <maxContacts value="64"/>
-    </gazebo>
-    <gazebo reference="rear_right_wheel">
+    <gazebo reference="limo${robot_id}/front_left_wheel">
+        <mu1>100</mu1>
+        <mu2>100</mu2>
+        <kp>10000000.0</kp>
+        <kd>1.0</kd>
+        <minDepth>0.01</minDepth>
+        <fdir1>1 0 0</fdir1>
+        <maxContacts value="64"/>
+    </gazebo>
+    <gazebo reference="limo${robot_id}/front_right_wheel">
+        <mu1>100</mu1>
+        <mu2>100</mu2>
+        <kp>10000000.0</kp>
+        <kd>1.0</kd>
+        <minDepth>0.01</minDepth>
+        <fdir1>1 0 0</fdir1>
+        <maxContacts value="64"/>
+    </gazebo>
+    <gazebo reference="limo${robot_id}/rear_left_wheel">
+        <mu1>100</mu1>
+        <mu2>100</mu2>
+        <kp>10000000.0</kp>
+        <kd>1.0</kd>
+        <minDepth>0.01</minDepth>
+        <fdir1>1 0 0</fdir1>
+        <maxContacts value="64"/>
+    </gazebo>
+    <gazebo reference="limo${robot_id}/rear_right_wheel">
         <mu1>100</mu1>
         <mu2>100</mu2>
@@ -222,19 +224,19 @@
         <update_rate>50</update_rate>
         <num_wheel_pairs>2</num_wheel_pairs>
-        <left_joint>front_left_wheel</left_joint>
-        <right_joint>front_right_wheel</right_joint>
-        <left_joint>rear_left_wheel</left_joint>
-        <right_joint>rear_right_wheel</right_joint>
+        <left_joint>limo${robot_id}/front_left_wheel</left_joint>
+        <right_joint>limo${robot_id}/front_right_wheel</right_joint>
+        <left_joint>limo${robot_id}/rear_left_wheel</left_joint>
+        <right_joint>limo${robot_id}/rear_right_wheel</right_joint>
         <wheel_separation>0.172</wheel_separation>
         <wheel_diameter>0.09</wheel_diameter>
         <max_wheel_torque>20</max_wheel_torque>
         <max_wheel_acceleration>1.0</max_wheel_acceleration>
-        <command_topic>cmd_vel</command_topic>
+        <command_topic>limo${robot_id}/cmd_vel</command_topic>
         <publish_odom>true</publish_odom>
         <publish_odom_tf>true</publish_odom_tf>
         <publish_wheel_tf>true</publish_wheel_tf>
-        <odometry_topic>odom</odometry_topic>
-        <odometry_frame>odom</odometry_frame>
-        <robot_base_frame>base_footprint</robot_base_frame>
+        <odometry_topic>limo${robot_id}/odom</odometry_topic>
+        <odometry_frame>limo${robot_id}/odom</odometry_frame>
+        <robot_base_frame>limo${robot_id}/base_footprint</robot_base_frame>
         <odometry_source>1</odometry_source>
         <ros>
@@ -243,3 +245,5 @@
         </plugin>
     </gazebo>
+    </xacro:macro>
+    <xacro:limo robot_id="$(arg robot_id)" />
 </robot>
